File: 8hp-board-phase.brd (EAGLE design)
At the start: 37.8 x 116.8 mm, 31 parts, among them IC1 TL074D, IC2 7805L, U2 MCP4822

Commit message: Add files via upload
Parts:
- removed R28, R29, R30: 10k, rcl:M0805
- added R5, R6, R8: 10k, rcl:M0805
- added S1: D6_PUSH_SWITCH, MusicThingModular:D6_PUSH_SWITCH
- moved R4 41.6 mm to (3.81, 74.9)
- moved IC1 29.2 mm to (7.62, 81.3)
- moved C15 17.3 mm to (8.89, 87.6)
- moved R1 17.1 mm to (16.5, 105.4)
- moved C16 12.8 mm to (8.89, 91.4)
- moved R2 6.84 mm to (3.81, 91.4)
- moved R3 6.35 mm to (3.81, 87.6)
- flipped ARDUINO_NANO1 to the bottom
- flipped SV1 to the bottom
- flipped SV7 to the bottom
- renumbered R25 to R7
Connections:
- new net D5: ARDUINO_NANO1.23, S1.P$3, S1.P$4
- net CVA1: now also R3.2; no longer R2.2
- net CVB: now also R1.1; no longer R4.1
- net GND: now also R6.1, S1.P$1, S1.P$2; no longer R1.1
- net N$1: now also R2.2, R3.1; no longer R2.1, R3.2
- net N$3: now also R1.2; no longer R4.2
- net N$72: now also R8.1; no longer R28.1
- net N$73: now also R5.1, R8.2; no longer R28.2, R29.1
- net N$75: now also R4.1, R5.2; no longer R29.2, R30.1
- net N$76: now also R4.2; no longer R30.2
- net PT: now also R6.2; no longer R1.2
- net PT2: now also R2.1; no longer R3.1
Routing:
- net N$73: track 15.5 -> 105.7 mm, vias 0 -> 2
- net D5: track 0.00 -> 84.1 mm, vias 0 -> 1
- net GND: track 244.8 -> 318.3 mm, vias 1 -> 7
- net N$76: track 143.5 -> 94.5 mm, vias 2 -> 4
- net 5V: track 119.4 -> 159.7 mm, vias 3 -> 5
- net AUDIO_IN: track 101.5 -> 66.8 mm, vias 4 -> 6
- net PT2: track 39.3 -> 67.6 mm, vias 1 -> 2
- net N$1: track 34.5 -> 7.70 mm, vias 2 -> 0
- net PT: track 73.8 -> 51.9 mm, vias 2 -> 4
- net D10: track 9.35 -> 27.5 mm, vias 1 -> 2
- net N$21: track 99.5 -> 82.8 mm, vias 3 -> 4
- net N$72: track 47.3 -> 32.1 mm, vias 2 -> 1
- net D11: track 9.35 -> 24.3 mm, vias 1 -> 2
- net -12V: track 142.9 -> 128.0 mm, vias 2 -> 8
- net +12V: track 131.4 -> 142.7 mm, vias 2 -> 7
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- added copper zone on layer 1, net GND
- added copper zone on layer 16, net GND
