File: 8hp-board-phase.sch (EAGLE design)
At the start: 31 parts, among them IC1 TL074D, IC2 7805L, U2 MCP4822

Commit message: Add files via upload
Parts:
- removed R30: 10k, rcl:R-EU_M0805
- added R6: 10k, rcl:R-EU_M0805
- added S1: D6_PUSH_SWITCH, MusicThingModular:D6_PUSH_SWITCH
- renumbered R25 to R7, R28 to R8, R29 to R5
Connections:
- new net D5: ARDUINO_NANO1.D5, S1.P
- net CVA1: now also R3.2; no longer R2.2
- net CVB: now also R1.1; no longer R4.1
- net GND: now also R6.1, S1.O; no longer R1.1
- net N$1: now also R2.2, R3.1; no longer R2.1, R3.2
- net N$3: now also R1.2; no longer R4.2
- net N$75: now also R4.1; no longer R30.1
- net N$76: now also R4.2; no longer R30.2
- net PT: now also R6.2; no longer R1.2
- net PT2: now also R2.1; no longer R3.1
Other:
- moved on the sheet: R1, R2, R3, R4
